File: PCB/Project Lab 3 BMS.kicad_pcb (KiCad board)
At the start: 2 copper layers, 46 parts, among them J1 Conn_01x02, J3 Conn_01x06, Q1 IRLR7843, Q2 IRLR7843, Q3 PMOS, SW1 Start Swtich, U1 BQ76920PW, U3 ESP32-DEVKIT-V1

Commit message: Update
Parts:
- removed J3: Conn_01x06, Connector_JST:JST_XH_B6B-XH-A_1x06_P2.50mm_Vertical
- removed R17, R18, R21: 1k, Resistor_SMD:R_0805_2012Metric
- removed R5, R6, R7: 1k, Capacitor_SMD:C_0805_2012Metric
- added J2: Conn_01x06, Connector_JST:JST_XH_B6B-XH-A_1x06_P2.50mm_Vertical, F.Cu at (30.5, 59.5)
- added RBAT+1: 1k, Resistor_SMD:R_0805_2012Metric, F.Cu at (145.1, 97.3)
- added RBAT-1: 1k, Resistor_SMD:R_0805_2012Metric, F.Cu at (145.1, 100.3)
- added RCELL1: 1k, Capacitor_SMD:C_0805_2012Metric, F.Cu at (140.7, 103.5)
- added RCELL2: 1k, Capacitor_SMD:C_0805_2012Metric, F.Cu at (140.7, 106.5)
- added RCELL3: 1k, Capacitor_SMD:C_0805_2012Metric, F.Cu at (140.7, 109.5)
- added RCELL4: 1k, Resistor_SMD:R_0805_2012Metric, F.Cu at (145.1, 103.2)
- moved U3 188.7 mm to (31.5, 165.0)
- moved J1 124.4 mm to (146.4, 113.9), turned to 0 degrees
- moved C8 88.7 mm to (153.2, 62.2)
- moved D2 82.1 mm to (151.9, 64.7)
- moved D1 72.4 mm to (150.2, 99.7)
- moved D4 72.4 mm to (150.2, 103.0)
- moved Q1 55.6 mm to (145.2, 64.7)
- moved Q2 55.6 mm to (145.2, 72.9)
- moved Q3 55.6 mm to (145.2, 81.1)
- moved R10 55.6 mm to (133.9, 63.0)
- moved R11 55.6 mm to (133.9, 67.9)
- moved R13 55.6 mm to (133.9, 77.7)
- moved R14 55.6 mm to (133.9, 82.6)
- moved R15 55.6 mm to (133.9, 87.5)
- moved R12 55.6 mm to (133.9, 72.8)
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Connections:
- C12 pad 2: Net-(C12-Pad2) -> Net-(U1-VC4)
- C13 pad 1: Net-(C12-Pad2) -> Net-(U1-VC4)
- C13 pad 2: Net-(U1-VC4) -> Net-(U1-VC3)
- C3 pad 1: Net-(U1-VC4) -> Net-(U1-VC3)
- C3 pad 2: Net-(U1-VC3) -> Net-(U1-VC2)
- C4 pad 1: Net-(U1-VC3) -> Net-(U1-VC2)
- C4 pad 2: Net-(U1-VC2) -> Net-(U1-VC1)
- C6 pad 1: Net-(U1-VC2) -> Net-(U1-VC1)
- U1 pad 16: unconnected-(U1-VC1-Pad16) -> Net-(U1-VC1)
