File: PCB/Project Lab 3 BMS.kicad_sch (KiCad schematic)
At the start: 37 parts, among them J1 Conn_01x04, J2 Screw_Terminal_01x02, Q1 CSD17571Q2T, Q2 CSD17571Q2T, U1 BQ76920PW, U2 ESP32-WROOM-32, U3 LD1086V33-DG

Commit message: update
Parts:
- removed F1: Fuse, symbol Device:Fuse
- removed J1: Conn_01x04, symbol Connector_Generic:Conn_01x04
- removed J2: Screw_Terminal_01x02, symbol Connector:Screw_Terminal_01x02
- removed R1, R4, R8: 100, symbol Device:R
- removed R9: 10, symbol Device:R
- removed RSHUNT1: 5M, symbol Device:R
- removed TH1: 10kNTC, symbol Device:Thermistor_US
- added C12, C13, C15, C19: 1uF, symbol Device:C_Small_US
- added C14: 7400pF, symbol Device:C
- added C16, C17, C18: 0.1uF, symbol Device:C_Small_US
- added D1, D4: D, symbol Device:D
- added D2: D_Schottky, symbol Device:D_Schottky
- added D3: SMCJ75AFS, symbol Device:D_TVS
- added J1: BATT+, symbol Connector_Generic:Conn_01x01
- added J2: BATT-, symbol Connector_Generic:Conn_01x01
- added J3: Conn_01x06, symbol Connector_Generic:Conn_01x06
- added R17, R18, R21: 1k, symbol Device:R
- added R19, R20: 100, symbol Device:R
- C1, C2, C5, C9: value 100nF -> 0.1uF
- C3, C4, C6, C7: value 100nF -> 1uF
- R10: value 1K -> 1k
- R12: value 10 -> 1k
- R14: value 1k -> R
- R16: value 10k -> 3k
- R5, R6, R7: value 100 -> 1k
Connections:
- net BAT: now also C8.1
- net BATT-: now also C10.2, C11.2, C7.2, C8.2, R14.2, R16.2, U1.3 (VSS), U2.1 (GND), U2.15 (GND), U2.38 (GND), U2.39 (GND), U3.1 (ADJ/GND), C14.2, C15.2, C17.2, C18.1, C19.1, D3.1 (A1), J3.6 (Pin_6), R20.2, R21.1; no longer C2.2, C5.2, C6.1, Q2.1 (D), R11.2, U1.17 (VC0)
- net DSG_GATE: now also Q1.2 (G), R11.1
- net REGOUT: no longer R16.2
- net SRN: now also C16.2, C17.1, R19.1
- net SRP: now also C16.1, C18.2, R20.1
- net at C9.1: now also C2.2, Q2.3 (S), R13.2, D2.2 (A), D4.2 (A); no longer C2.1
- net at C1.1: now also Q1.3 (S), R11.2, R14.1, R19.2; no longer C9.2
- net TS1: now reaches R16.1, U1.6 (TS1)
- net TS1: now also C14.1
- net at Q2.2 (G): now also R10.2, R13.1, D1.1 (K), D2.1 (K); no longer R11.1
- net CELL 3: now reaches R5.1
- net CELL 3: now also J3.3 (Pin_3)
- net CELL 2: now reaches R6.1
- net CELL 2: now also J3.4 (Pin_4)
- net at R7.1: no longer names the net of R7.1
- net at R7.1: now also J3.5 (Pin_5)
- net at R10.1: now also R12.2, D1.2 (A)
- net BATT+: now reaches U1.9 (REGSRC)
- net BATT+: now also C15.1; no longer R14.1
- removed net GND: C1.2, C10.2, C11.2, C7.2, C8.2, Q1.1 (D), R13.2, U1.3 (VSS), U2.1 (GND), U2.15 (GND), U2.38 (GND), U2.39 (GND), U3.1 (ADJ/GND)
- net VC1: no longer names the net of C4.2, R7.2
- net VC1: now also C6.1, U1.15 (VC2); no longer C5.1, U1.16 (VC1)
- net VC2: no longer names the net of C3.2, C4.1, R6.2
- net VC2: now also U1.14 (VC3); no longer U1.15 (VC2)
- net VC3: no longer names the net of C3.1, R5.2, U1.13 (VC4)
- net VC3: now also C13.2; no longer U1.12 (VC5), U1.14 (VC3)
- new net: C19.2, R21.2
- new net: C12.1, R18.2, U1.12 (VC5)
- new net: C1.2, C2.1
- new net: C5.2, D4.1 (K)
- new net: C5.1, C9.2
- new net: C12.2, C13.1, R17.2
- new net: Q1.1 (D), Q2.1 (D)
- new net BAT+: D3.2 (A2), J3.1 (Pin_1), R18.1
- new net CELL 4: J3.2 (Pin_2), R17.1
Other:
- note added: "OC/SHORT Sense"
- moved on the sheet: C6, C7, C8, Q1, Q2, R11, R13

Commit message: update again
Parts:
- added Q3: CSD17571Q2T, symbol Simulation_SPICE:NMOS
- R10: value 1k -> 1M
Connections:
- net BATT+: now also J1.1 (Pin_1)
- net BATT-: now also J2.1 (Pin_1), Q3.2 (G)
- net CHG_GATE: now also Q3.3 (S); no longer R12.1
- net at C19.2, R21.2: now also U1.17 (VC0)
- new net: Q3.1 (D), R12.1
Other:
- note added: "Voltage Regulator For ESP32"
- moved on the sheet: C1, C10, C11, C16, C17, C18, C2, C5, C8, C9, D1, D2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

Commit message: Update
Parts:
- removed J1: BATT+, symbol Connector_Generic:Conn_01x01
- removed J2: BATT-, symbol Connector_Generic:Conn_01x01
- added J1: Conn_01x02, symbol Connector_Generic:Conn_01x02
- added J2: Conn_01x06, symbol Connector_Generic:Conn_01x06
- R14: value R -> 1M
Connections:
- net BAT+: now also J2.1 (Pin_1)
- net BATT-: now also J2.6 (Pin_6)
- net CELL 2: now also J2.4 (Pin_4)
- net CELL 3: now also J2.3 (Pin_3)
- net CELL 4: now also J2.2 (Pin_2)
- net LOAD-: now reaches C2.2, C9.1, D2.2 (A), D4.2 (A), Q2.3 (S), R13.2
- net LOAD-: now also J1.2 (Pin_2)
- net at J3.5 (Pin_5), R7.1: now also J2.5 (Pin_5)
- net LOAD+: now reaches C5.2, D4.1 (K)
- net LOAD+: now also J1.1 (Pin_1)
Other:
- note added: "BAT+ to BAT pin"
- note added: "Output Connector (Charge/Discharge)"
- note added: "Voltage Regulator For ESP32 3.3v"
- note removed: "Voltage Regulator For ESP32"

Commit message: Update
Parts:
- removed C10, C11: 10uF, symbol Device:C_Small_US
- removed D2: D_Schottky, symbol Device:D_Schottky
- removed J2: Conn_01x06, symbol Connector_Generic:Conn_01x06
- removed Q3: CSD17571Q2T, symbol Simulation_SPICE:NMOS
- removed R16: 3k, symbol Device:R
- removed U3: LD1086V33-DG, Package_TO_SOT_THT:TO-220-3_Vertical, symbol Regulator_Linear:LD1086V33-DG
- added D2: D_Zener, symbol Device:D_Zener
- added Q3: PMOS, symbol Simulation_SPICE:PMOS
- added SW1: Start Swtich, symbol Switch:SW_Push
- added TH1: 10k, symbol Device:Thermistor
- D1: value D -> 1.25V
- D3: value SMCJ75AFS -> SMCJ45A
- Q1, Q2: value CSD17571Q2T -> IRLR7843
Connections:
- net BATT-: now also Q3.2 (G), SW1.1; no longer R21.1
- net CHG_GATE: now also Q3.3 (S)
- net LOAD-: now also D2.2 (A)
- net TS1: now also TH1.1
- net at D1.1 (K), Q2.2 (G), R10.2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: now also D2.1 (K)
- net at R12.1: now also Q3.1 (D)
- new net: SW1.2, TH1.2
- new net BAT-: R21.1
Other:
- note added: "FETS"
- note added: "Use Vishay WSL2512R0010FEA 1W power resistor"
- note removed: "Voltage Regulator For ESP32 3.3v"
- moved on the sheet: C1, C16, C17, C18, C2, C5, C9, D1, D4, J3, Q1, Q2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

Commit message: Footprints Assigned
Parts:
- removed U2: ESP32-WROOM-32, RF_Module:ESP32-WROOM-32, symbol RF_Module:ESP32-WROOM-32
- added U3: ESP32-DEVKIT-V1, Snapeda:MODULE_ESP32_DEVKIT_V1, symbol Snapeda:ESP32-DEVKIT-V1
- C1, C12, C13, C14, C15, C16, C17, C18, C19, C2, C3, C4, C5, C6, C7, C9, R2, R3, R5, R6, R7: footprint (none) -> Capacitor_SMD:C_0805_2012Metric
- C8: footprint (none) -> Capacitor_SMD:C_1206_3216Metric
- D1, D4: footprint (none) -> Diode_SMD:D_SOD-123
- D2: footprint (none) -> Diode_SMD:D_0201_0603Metric
- D3: footprint (none) -> Diode_SMD:D_SMC
- J1: footprint (none) -> TerminalBlock_Phoenix:TerminalBlock_Phoenix_MKDS-1,5-2_1x02_P5.00mm_Horizontal
- J3: footprint (none) -> Connector_JST:JST_XH_B6B-XH-A_1x06_P2.50mm_Vertical
- Q1, Q2, Q3: footprint (none) -> Package_TO_SOT_SMD:TO-252-2
- R10, R11, R12, R13, R14, R15: footprint (none) -> Resistor_SMD:R_2512_6332Metric
- R17, R18, R19, R20, R21, TH1: footprint (none) -> Resistor_SMD:R_0805_2012Metric
- SW1: footprint (none) -> Button_Switch_SMD:SW_SPST_PTS645Sx43SMTR92
Connections:
- net ALERT: now also U3.4 (D2)
- net BATT-: now also U3.2 (GND), U3.29 (GND)
- net SCL: now also U3.11 (D21)
- net SDA: now also U3.14 (D22)
Other:
- note added: "ESP32"
- moved on the sheet: C8, J1

Commit message: Update
Parts:
- removed J3: Conn_01x06, Connector_JST:JST_XH_B6B-XH-A_1x06_P2.50mm_Vertical, symbol Connector_Generic:Conn_01x06
- added J2: Conn_01x06, Connector_JST:JST_XH_B6B-XH-A_1x06_P2.50mm_Vertical, symbol Connector_Generic:Conn_01x06
- renumbered R18 to RBAT+1, R21 to RBAT-1, R7 to RCELL1, R6 to RCELL2, R5 to RCELL3, R17 to RCELL4
Connections:
- net BAT- is gone; now on net BATT-: RBAT-1.1
- net BAT+: now also J2.1 (Pin_1)
- net BATT-: now also J2.6 (Pin_6)
- net CELL 2: now also J2.4 (Pin_4)
- net CELL 3: now also J2.3 (Pin_3)
- net CELL 4: now also J2.2 (Pin_2)
- net at C3.2, C4.1, RCELL2.2: now also U1.15 (VC2); no longer U1.14 (VC3)
- net at C4.2, C6.1, RCELL1.2: now also U1.16 (VC1); no longer U1.15 (VC2)
- net at C13.2, C3.1, RCELL3.2: now also U1.14 (VC3); no longer U1.13 (VC4)
- net at RCELL1.1: now also J2.5 (Pin_5)
- net at C12.2, C13.1, RCELL4.2: now also U1.13 (VC4)
