File: PCB/Project Lab 3 BMS.kicad_sch (KiCad schematic)
At the start: 46 parts, among them J1 Conn_01x02, J2 Conn_01x06, Q1 IRLR7843, Q2 IRLR7843, Q3 PMOS, SW1 Start Swtich, U1 BQ76920PW, U3 ESP32-DEVKIT-V1

Commit message: Changed IC for Monitoring
Parts:
- removed C1, C16, C17, C18, C2, C5, C9: 0.1uF, Capacitor_SMD:C_0805_2012Metric, symbol Device:C_Small_US
- removed C14: 7400pF, Capacitor_SMD:C_0805_2012Metric, symbol Device:C
- removed C15, C19, C3, C4, C6, C7: 1uF, Capacitor_SMD:C_0805_2012Metric, symbol Device:C_Small_US
- removed C8: 4.7uF, Capacitor_SMD:C_1206_3216Metric, symbol Device:C_Small_US
- removed D1: 1.25V, Diode_SMD:D_SOD-123, symbol Device:D
- removed D2: D_Zener, Diode_SMD:D_0201_0603Metric, symbol Device:D_Zener
- removed D3: SMCJ45A, Diode_SMD:D_SMC, symbol Device:D_TVS
- removed D4: D, Diode_SMD:D_SOD-123, symbol Device:D
- removed J1: Conn_01x02, TerminalBlock_Phoenix:TerminalBlock_Phoenix_MKDS-1,5-2_1x02_P5.00mm_Horizontal, symbol Connector_Generic:Conn_01x02
- removed J2: Conn_01x06, Connector_JST:JST_XH_B6B-XH-A_1x06_P2.50mm_Vertical, symbol Connector_Generic:Conn_01x06
- removed Q1, Q2: IRLR7843, Package_TO_SOT_SMD:TO-252-2, symbol Simulation_SPICE:NMOS
- removed Q3: PMOS, Package_TO_SOT_SMD:TO-252-2, symbol Simulation_SPICE:PMOS
- removed R10, R11, R13, R14, R15: 1M, Resistor_SMD:R_2512_6332Metric, symbol Device:R
- removed R12: 1k, Resistor_SMD:R_2512_6332Metric, symbol Device:R
- removed R19, R20: 100, Resistor_SMD:R_0805_2012Metric, symbol Device:R
- removed R2, R3: 4.7k, Capacitor_SMD:C_0805_2012Metric, symbol Device:R
- removed RBAT+1, RBAT-1, RCELL4: 1k, Resistor_SMD:R_0805_2012Metric, symbol Device:R
- removed RCELL1, RCELL2, RCELL3: 1k, Capacitor_SMD:C_0805_2012Metric, symbol Device:R
- removed SW1: Start Swtich, Button_Switch_SMD:SW_SPST_PTS645Sx43SMTR92, symbol Switch:SW_Push
- removed TH1: 10k, Resistor_SMD:R_0805_2012Metric, symbol Device:Thermistor
- removed U1: BQ76920PW, Package_SO:TSSOP-20_4.4x6.5mm_P0.65mm, symbol Battery_Management:BQ76920PW
- added C10, C11: 10nF, symbol Device:C_Small_US
- added D5, D6, D7, D8: 9.1V, symbol Device:D_Zener
- added Q4, Q5, Q6, Q7: NMOS, symbol Simulation_SPICE:NMOS
- added R1: R, symbol Device:R
- added R16, R21, R24, R9: R_Dis, symbol Device:R
- added R17, R22, R25, R7: 1k, symbol Device:R
- added R18, R23, R26, R8: 100, symbol Device:R
- added U2: LTC6810HG-1-3ZZPBF, 05-08-1754_ADI, symbol LTC6810-1:LTC6810HG-1-3ZZPBF
- C12, C13: value 1uF -> 10nF; footprint Capacitor_SMD:C_0805_2012Metric -> (none)
Connections:
- net BATT- is gone; now on net GND: U3.2 (GND), U3.29 (GND)
- net GND: now reaches C13.2
- net GND: now also C12.2, C10.2, C11.2, D5.2 (A), D6.2 (A), D7.2 (A), D8.2 (A), Q4.3 (S), Q5.3 (S), Q6.3 (S), Q7.3 (S), R1.1, R16.2, R17.1, R18.1, R21.2, R22.1, R23.1, R24.2, R25.1, R26.1, R7.1, R8.1, R9.2, U2.21 (V-), U2.22 (V-), U2.23 (V-), U2.24 (V-), U2.28 (V-), U2.29 (V-)
- net C2: now reaches C12.1
- net C2: now also R23.2, U2.12 (C2)
- net C3: now reaches C13.1
- net C3: now also R26.2, U2.10 (C3); no longer C12.2
- net ALERT: no longer names the net of U3.4 (D2)
- net SCL: no longer names the net of U3.11 (D21)
- net SDA: no longer names the net of U3.14 (D22)
- new net: Q4.1 (D), R9.1
- new net: Q6.1 (D), R21.1
- new net: Q5.1 (D), R16.1
- new net: R1.2, U2.4 (C6), U2.5 (S6), U2.6 (C5), U2.7 (S5), U2.8 (C4), U2.9 (S4)
- new net: U2.1 (V-), U2.40 (SDO(NC)), U2.41 (SDI(NC)), U2.43 (V-), U2.44 (V-)
- new net: Q7.1 (D), R24.1
- new net C0: C10.1, R8.2, U2.16 (C0)
- new net C1: C11.1, R18.2, U2.14 (C1)
- new net S0: D5.1 (K), Q4.2 (G), R7.2, U2.17 (S0)
- new net S1: D6.1 (K), Q5.2 (G), R17.2, U2.15 (S1)
- new net S2: D7.1 (K), Q6.2 (G), R22.2, U2.13 (S2)
- new net S3: D8.1 (K), Q7.2 (G), R25.2, U2.11 (S3)
Other:
- note added: "Cell Balancing FETS"
- note removed: "BAT+ to BAT pin"
- note removed: "FETS"
- note removed: "OC/SHORT Sense"
- note removed: "Output Connector (Charge/Discharge)"
- note removed: "Use Vishay WSL2512R0010FEA 1W power resistor"
- moved on the sheet: U3

Commit message: update
Parts:
- removed Q4, Q5, Q6, Q7: NMOS, symbol Simulation_SPICE:NMOS
- removed U2: LTC6810HG-1-3ZZPBF, 05-08-1754_ADI, symbol LTC6810-1:LTC6810HG-1-3ZZPBF
- added C1: 4.7uF, symbol Device:C_Small_US
- added C14, C3: 10nF, symbol Device:C_Small_US
- added C2: 0.1uF, symbol Device:C_Small_US
- added C4, C5, C6, C7: 100nF, symbol Device:C_Small_US
- added J1: Conn_01x04, symbol Connector_Generic:Conn_01x04
- added Q1, Q2, Q3, Q4: 2N7002, Package_TO_SOT_SMD:SOT-23, symbol Transistor_FET:2N7002
- added R10, R2, R3, R4, R5, R6: R, symbol Device:R
- added TH1, TH2, TH3, TH4: Thermistor, symbol Device:Thermistor
- added U1: LTC6810HG-2-3ZZPBF, SSOP44G_05-08-1754_ADI, symbol LTC6810-2:LTC6810HG-2-3ZZPBF
- added U2: LT8610, Package_SO:MSOP-16-1EP_3x4.039mm_P0.5mm_EP1.651x2.845mm_ThermalVias, symbol Regulator_Switching:LT8610
- R1: value R -> 100
Connections:
- net C3: now also R1.1, C2.2; no longer C13.1, R26.2
- net S0: now also Q4.1 (G), U1.17 (S0)
- net S1: now also Q3.1 (G), U1.15 (S1)
- net S2: now also Q2.1 (G), U1.13 (S2)
- net S3: now also Q1.1 (G), U1.11 (S3)
- net at R9.1: now also Q4.3 (D)
- net at R21.1: now also Q2.3 (D)
- net SCK: now reaches U3.9 (D18)
- net at R16.1: now also Q3.3 (D)
- net V+: now reaches R1.2
- net V+: now also C3.2
- net at R24.1: now also Q1.3 (D)
- net C0: no longer names the net of C10.1, R8.2
- net C0: now also C7.2, U1.16 (C0)
- net C1: no longer names the net of C11.1, R18.2
- net C1: now also C6.2, U1.14 (C1)
- net C2: no longer names the net of C12.1, R23.2
- net C2: now also C5.2, U1.12 (C2)
- net GND renamed BAT-
- net BAT-: now also C1.1, C1.2, C14.2, C2.1, C3.1, C4.1, C5.1, C6.1, C7.1, J1.1 (Pin_1), J1.2 (Pin_2), J1.3 (Pin_3), Q1.2 (S), Q2.2 (S), Q3.2 (S), Q4.2 (S), R10.1, R6.1, TH1.2, TH2.2, TH3.2, TH4.2, U1.21 (V-*), U1.22 (V-*), U1.23 (V-*), U1.24 (V-*), U1.27 (ISOMD), U1.28 (V-), U1.29 (V-), U2.17 (GND), U2.4 (EN/UV), U2.5 (VIN), U2.6 (VIN), U2.7 (GND), U2.8 (GND); no longer R1.1
- new net: R2.1, R3.1, R4.1, R5.1
- new net: C13.1, C4.2, R26.2, U1.10 (C3)
- new net: U2.10 (SW), U2.11 (SW), U2.9 (SW)
- new net: R5.2, TH4.1
- new net: R6.2, U1.4 (C6), U1.6 (C5), U1.8 (C4)
- new net: C14.1, R10.2, U1.3 (V+)
- new net BATT- : J1.4 (Pin_4)
- new net GPIO1: R2.2, TH1.1, U1.18 (GPIO1)
- new net GPIO2: R3.2, TH2.1, U1.19 (GPIO2)
- new net GPIO3: R4.2, TH3.1, U1.20 (GPIO3)
Other:
- note added: "Connector"
