File: PCB/Project Lab 3 BMS.kicad_sch (KiCad schematic)
At the start: 47 parts, among them J1 Conn_01x04, Q1 2N7002, Q2 2N7002, Q3 2N7002, Q4 2N7002, U1 LTC6810HG-2-3ZZPBF, U2 LT8610, U3 ESP32-DEVKIT-V1

Commit message: Footprint
Parts:
- removed R5: R, symbol Device:R
- removed TH4: Thermistor, symbol Device:Thermistor
- C2, C3, C4, C5, C6, C7: footprint (none) -> Capacitor_SMD:C_1206_3216Metric_Pad1.33x1.80mm_HandSolder
- R16, R17, R21, R22, R24, R25, R7, R8, R9: footprint (none) -> Resistor_SMD:R_1206_3216Metric_Pad1.30x1.75mm_HandSolder
Connections:
- net VREF2: now reaches R2.1, R3.1, R4.1
- no-connect marks 0 -> 2
Other:
- note removed: "Cell Balancing FETS"
- moved on the sheet: C1, C14, C4, C5, C6, C7, R10, R6, U1

Commit message: Serial IC Updates
Parts:
- added Q5: NPN, symbol Simulation_SPICE:NPN
- added R5: 10R, symbol Device:R
- R10: value R -> 100R
Connections:
- net BAT-: no longer C1.1, J1.1 (Pin_1), R10.1, R24.2, R26.1, U2.4 (EN/UV), U2.5 (VIN), U2.6 (VIN)
- net at U1.1 (V-*): now also U1.40 (SDO(IBIAS)**), U1.41 (SDI(ICMP)**), U1.43 (V-*), U1.44 (V-*)
- net at U1.32 (VREG): now also Q5.3 (E)
- new net: Q5.2 (B), R5.2
- new net Bat+: C1.1, J1.1 (Pin_1), Q5.1 (C), R10.1, R24.2, R26.1, U2.4 (EN/UV), U2.5 (VIN), U2.6 (VIN)
- no-connect marks 2 -> 4
Other:
- moved on the sheet: C1, C14, C4, C5, C6, C7, R10, R6, U1, U2
