File: Power Systems/Power Systems.kicad_sch (KiCad schematic)
At the start: 66 parts, among them IC1 INA296A3IDDFR, J5 Conn_01x19, J6 Conn_01x19, J8 Conn_01x02, J9 Conn_01x02, Q19 IRLR7843, Q20 PMOS, Q21 IRLR7843, Q22 NMOS, Q23 NMOS, Q24 NMOS, Q25 NMOS, U21 ESP32-DEVKIT-V1, U22 LM2596S-3.3, U23 LM2596S-5, U24 LTC6810HG-1-3ZZPBF

Commit message: Serial Comms IC Updates
Parts:
- removed C43, C44, C45, C46: 10nF, Capacitor_SMD:C_0805_2012Metric, symbol Device:C_Small_US
- removed D18, D19, D20, D21: 9.1V, symbol Device:D_Zener
- removed IC1: INA296A3IDDFR, ESP32 Dev Kit:SOT65P280X110-8N, symbol myLibrary:INA296A3IDDFR
- removed Q22, Q23, Q24, Q25: NMOS, symbol Simulation_SPICE:NMOS
- removed R81: R, symbol Device:R
- removed R82, R83, R84, R85: R_Dis, Resistor_SMD:R_1206_3216Metric, symbol Device:R
- removed R86, R87, R88, R89: 1k, Resistor_SMD:R_1206_3216Metric, symbol Device:R
- removed R90, R91, R92, R93: 100, Resistor_SMD:R_1206_3216Metric, symbol Device:R
- removed U24: LTC6810HG-1-3ZZPBF, 05-08-1754_ADI, symbol LTC6810-1:LTC6810HG-1-3ZZPBF
- added BT1, BT2, BT3: Battery_Cell, symbol Device:Battery_Cell
- added C4, C5, C6, C7: 1nF, symbol Device:C_Small_US
- added Q3, Q4, Q5: AO3400A, Package_TO_SOT_SMD:SOT-23, symbol Transistor_FET:AO3400A
- added R10, R8, R9: 220R, symbol Device:R
- added R11, R12, R13: 100kR, symbol Device:R
- added R14: 40R, symbol Device:R
- added R15: 1MR, symbol Device:R
- added R4, R5, R6, R7: 43R, symbol Device:R
- added SW1: SW_Push, symbol Switch:SW_Push
- added U2: INA226, Package_SO:TSSOP-10_3x3mm_P0.5mm, symbol Sensor_Energy:INA226
- added U3: BQ76920PW, Package_SO:TSSOP-20_4.4x6.5mm_P0.65mm, symbol Battery_Management:BQ76920PW
Connections:
- net 3.3v: now also U2.6 (VS)
- net CELL 1: now also BT1.1 (+), BT2.2 (-), R6.1
- net CELL 2: now also BT2.1 (+), BT3.2 (-), R5.1
- net GND: now also BT1.2 (-), BT3.1 (+), C7.2, R15.2, R4.1, R7.1, U2.1 (A1), U2.2 (A0), U2.7 (GND), U3.14 (VC3), U3.17 (VC0), U3.3 (VSS)
- net SCL: now also U2.5 (SCL), U3.5 (SCL)
- net SDA: now also U2.4 (SDA), U3.4 (SDA)
- net SRN: now also U2.8 (Vbus), U2.9 (Vin-)
- net SRP: now also U2.10 (Vin+)
- new net: Q4.1 (G), R12.1, R9.1
- new net: R15.1, SW1.1
- new net: C5.1, C6.2, Q4.2 (S), Q5.3 (D), R13.2, R5.2
- new net: C7.1, U3.7 (CAP1)
- new net: SW1.2, U3.6 (TS1)
- new net: Q3.1 (G), R10.1, R11.1
- new net: C4.2, Q3.3 (D), R11.2, R7.2
- new net: Q5.1 (G), R13.1, R8.1
- new net: C4.1, C5.2, Q3.2 (S), Q4.3 (D), R12.2, R6.2
- new net: C6.1, Q5.2 (S), R4.2
- new net: R14.1, U3.10 (BAT)
- new net: U3.18 (SRP), U3.19 (SRN)
- new net VC1: R10.2, U3.16 (VC1)
- new net VC2: R9.2, U3.15 (VC2)
- new net VC3: R8.2
- no-connect marks 12 -> 15
Other:
- note added: "Cell Monitoring IC"
- note added: "I2C Address @ 0x40 with A1/A0 Configuration"
- note added: "Passive Cell Balancing"
- note removed: "Cell Balancing FETS"
